Commit message: add top plate dae

File: gki_turtlebot/gki_turtlebot_description/urdf/stacks/hexagons_freiburg.urdf.xacro (robot description, xacro)
@@ -206,5 +206,5 @@
         <origin xyz="0 0 0" rpy="0 0 0"/>
         <geometry>
-          <mesh filename="package://gki_turtlebot_description/meshes/stacks/hexagons_freiburg/plate_top.stl"/>
+          <mesh filename="package://gki_turtlebot_description/meshes/stacks/hexagons_freiburg/plate_top.dae"/>
         </geometry>
         <material name="Grey">
