Commit message: adjusted origin for base_laser

File: gki_turtlebot/gki_sensors_description/urdf/hokuyo_urg.urdf.xacro (robot description, xacro)
@@ -7,9 +7,15 @@
   >
     <xacro:macro name="hokuyo_urg" params="name parent *origin ros_topic update_rate ray_count min_angle max_angle">
-      <joint name="${name}_joint" type="fixed">
+      <joint name="${name}_base_joint" type="fixed">
         <insert_block name="origin" />
         <parent link="${parent}"/>
+        <child link="${name}_base_link"/>
+      </joint>
+      <joint name="${name}_joint" type="fixed">
+        <origin xyz="0 0 0.056" rpy="0 0 0" />
+        <parent link="${name}_base_link"/>
         <child link="${name}_link"/>
       </joint>
+      <link name="${name}_base_link" />
       <link name="${name}_link">
         <inertial>
@@ -19,5 +25,5 @@
         </inertial>
         <visual>
-          <origin xyz="0 0 0" rpy="0 0 0" />
+          <origin xyz="0 0 -0.056" rpy="0 0 0" />
           <geometry>
           <mesh filename="package://gki_sensors_description/meshes/hokuyo_urg$(optenv TEST_SELF_FILTER).dae"/>
@@ -25,5 +31,5 @@
         </visual>
         <collision>
-          <origin xyz="0 0 -0.0115" rpy="0 0 0" />
+          <origin xyz="0 0 -0.021" rpy="0 0 0" />
           <geometry>
           <box size="0.05 0.05 0.07" />
