Commit message: add axis joints to urdf

File: gki_turtlebot/gki_sensors_description/urdf/axis215.urdf.xacro (robot description, xacro)
@@ -32,4 +32,30 @@
         </collision>
       </link>
+      <link name="${name}_panned_link" />
+      <link name="${name}_tilted_link" />
+      <link name="${name}_optical_link" />
+      <joint name="${name}_pan" type="revolute">
+          <!-- TODO check height of actual camera to camera base -->
+          <origin xyz="0.0 0.0 0.05" rpy="0.0 0.0 -1.57079632679489661922" />
+          <axis xyz="0 0 1" />
+          <parent link="${name}_link"/>
+          <child link="${name}_panned_link"/>
+          <limit lower="-3.14" upper="3.14" effort="1.0" velocity="3.14" />
+      </joint>
+      <joint name="${name}_tilt" type="revolute">
+          <axis xyz="0 -1 0" />
+          <parent link="${name}_panned_link"/>
+          <child link="${name}_tilted_link"/>
+          <limit lower="0.0" upper="1.57079632679489661922" effort="1.0" velocity="3.14" />
+      </joint>
+      <!-- If optical frame is somewhat turned, put this here -->
+      <joint name="${name}_tilt_to_optical" type="fixed">
+          <origin xyz="0.0 0.0 0.0" rpy="0.0 0.0 0.0" />
+          <parent link="${name}_tilted_link"/>
+          <child link="${name}_optical_link"/>
+      </joint>
+      <!-- axis_link is base/center of camera???
+           Finally: make sure that frame is send in axis_camera pubs for imgs and everything that has a header -->
+    <!-- Also needs to be tested for offsets/rotation + direction -->
     </xacro:macro>
 </robot>

File: gki_zerg/gki_zerg_description/robot/zerg.urdf.xacro (robot description, xacro)
@@ -19,5 +19,4 @@
   </xacro:axis215>
   <joint name="imu_joint" type="fixed">
-      <axis xyz="0 1 0"/>
       <origin xyz="0.056 0.062 0.0202" rpy="0 0 0"/>
       <parent link="base_link"/>

Commit message: fixed axis tf

File: gki_turtlebot/gki_sensors_description/urdf/axis215.urdf.xacro (robot description, xacro)
@@ -36,7 +36,6 @@
       <link name="${name}_optical_link" />
       <joint name="${name}_pan" type="revolute">
-          <!-- TODO check height of actual camera to camera base -->
-          <origin xyz="0.0 0.0 0.05" rpy="0.0 0.0 -1.57079632679489661922" />
-          <axis xyz="0 0 1" />
+          <origin xyz="0.0 0.0 0.09" rpy="0.0 0.0 -1.57079632679489661922" />
+          <axis xyz="0 0 -1" />
           <parent link="${name}_link"/>
           <child link="${name}_panned_link"/>

File: gki_zerg/gki_zerg_description/urdf/zerg_base.urdf.xacro (robot description, xacro)
@@ -72,5 +72,5 @@
     <zerg_wheel link_name="wheel_rear_left_link" />
     <zerg_wheel link_name="wheel_rear_right_link" />
-    <joint name="wheel_front_left_joint" type="continuous">
+    <joint name="wheel_front_left_joint" type="fixed">
       <parent link="base_link"/>
       <child link="wheel_front_left_link"/>
@@ -78,5 +78,5 @@
       <axis xyz="0 0 1"/>
     </joint>
-    <joint name="wheel_front_right_joint" type="continuous">
+    <joint name="wheel_front_right_joint" type="fixed">
       <parent link="base_link"/>
       <child link="wheel_front_right_link"/>
@@ -84,5 +84,5 @@
       <axis xyz="0 0 1"/>
     </joint>
-    <joint name="wheel_rear_left_joint" type="continuous">
+    <joint name="wheel_rear_left_joint" type="fixed">
       <parent link="base_link"/>
       <child link="wheel_rear_left_link"/>
@@ -90,5 +90,5 @@
       <axis xyz="0 0 1"/>
     </joint>
-    <joint name="wheel_rear_right_joint" type="continuous">
+    <joint name="wheel_rear_right_joint" type="fixed">
       <parent link="base_link"/>
       <child link="wheel_rear_right_link"/>

Commit message: fixed rotation between axis tilt and optical link

File: gki_turtlebot/gki_sensors_description/urdf/axis215.urdf.xacro (robot description, xacro)
@@ -50,5 +50,5 @@
       <!-- If optical frame is somewhat turned, put this here -->
       <joint name="${name}_tilt_to_optical" type="fixed">
-          <origin xyz="0.0 0.0 0.0" rpy="0.0 0.0 0.0" />
+          <origin xyz="0.0 0.0 0.0" rpy="${-M_PI/2} 0 ${-M_PI/2}" />
           <parent link="${name}_tilted_link"/>
           <child link="${name}_optical_link"/>
