Commit message: hokuyo_urg.xacro

File: gki_turtlebot/gki_turtlebot_description/robots/kobuki_hexagons_freiburg_kinect.urdf.xacro (robot description, xacro)
@@ -15,3 +15,7 @@
   <stack_hexagons_freiburg parent="base_link"/>
   <sensor_kinect  parent="base_link"/>
+  <include filename="$(find gki_sensors_description)/urdf/hokuyo_urg.urdf.xacro" />
+  <xacro:hokuyo_urg name="base_laser" parent="plate_middle_link" ros_topic="base_scan" update_rate="10" ray_count="667" min_angle="120" max_angle="-120">
+    <origin xyz="-0.04 0.0 0.008" rpy="0 0 0"/>
+  </xacro:hokuyo_urg>
 </robot>

Commit message: add base_footprint to urdf

File: gki_turtlebot/gki_turtlebot_description/robots/kobuki_hexagons_freiburg_kinect.urdf.xacro (robot description, xacro)
@@ -14,4 +14,11 @@
   <kobuki/>
   <stack_hexagons_freiburg parent="base_link"/>
+  <!-- base_footprint is a fictitious link(frame) that is on the ground right below base_link origin, navigation stack depends on this frame -->
+  <link name="base_footprint" />
+  <joint name="base_footprint_joint" type="fixed">
+    <origin xyz="0 0 0.017" rpy="0 0 0" />
+    <parent link="base_footprint"/>
+    <child link="base_link" />
+  </joint>
   <sensor_kinect  parent="base_link"/>
   <include filename="$(find gki_sensors_description)/urdf/hokuyo_urg.urdf.xacro" />

Commit message: removed base_link from kobuki_hexagons_freiburg_kinect (already in         kobuki)

File: gki_turtlebot/gki_turtlebot_description/robots/kobuki_hexagons_freiburg_kinect.urdf.xacro (robot description, xacro)
@@ -14,11 +14,4 @@
   <kobuki/>
   <stack_hexagons_freiburg parent="base_link"/>
-  <!-- base_footprint is a fictitious link(frame) that is on the ground right below base_link origin, navigation stack depends on this frame -->
-  <link name="base_footprint" />
-  <joint name="base_footprint_joint" type="fixed">
-    <origin xyz="0 0 0.017" rpy="0 0 0" />
-    <parent link="base_footprint"/>
-    <child link="base_link" />
-  </joint>
   <sensor_kinect  parent="base_link"/>
   <include filename="$(find gki_sensors_description)/urdf/hokuyo_urg.urdf.xacro" />
