Commit message: add axis model

File: gki_zerg/gki_zerg_description/robots/zerg.urdf.xacro (robot description, xacro)
@@ -11,7 +11,11 @@
   <zerg_parts parent="base_link"/>
   <include filename="$(find gki_sensors_description)/urdf/hokuyo_urg.urdf.xacro" />
+  <include filename="$(find gki_sensors_description)/urdf/axis215.urdf.xacro" />
   <xacro:hokuyo_urg name="base_laser" parent="base_link" ros_topic="base_scan" update_rate="10" ray_count="667" min_angle="120" max_angle="-120">
     <origin xyz="0.1 0.0 0.138" rpy="0 0 0"/>
   </xacro:hokuyo_urg>
+  <xacro:axis215 name="axis" parent="base_link">
+    <origin xyz="0.0 0.0 0.41" rpy="0 0 0"/>
+  </xacro:axis215>
   <joint name="imu_joint" type="fixed">
       <axis xyz="0 1 0"/>

File: gki_zerg/gki_zerg_description/urdf/zerg_parts.urdf.xacro (robot description, xacro)
@@ -55,5 +55,5 @@
         <origin xyz="0 0 0" rpy="0 0 0"/>
         <geometry>
-            <box size="0.04 0.02 0.435" />
+            <box size="0.04 0.357 0.02" />
         </geometry>
       </collision>
