Commit message: adjusted the angle of the front camera

File: gki_zerg/gki_zerg_description/urdf/front_cam.urdf.xacro (robot description, xacro)
@@ -35,5 +35,5 @@
       </joint>
       <joint name="${name}_tilt" type="fixed">
-          <origin xyz="0.0 0.0 0.0" rpy="0.0 -0.3 0.0" />
+          <origin xyz="0.0 0.0 0.0" rpy="0.0 0.0 0.0" />
           <parent link="${name}_panned_link"/>
           <child link="${name}_tilted_link"/>
