Commit message: changed urdf to represent zerg sickrd configuration, added cube holder model for rviz, added device argument to logitech_teleop.lauch to fix compatibility for simulation

File: gki_zerg/gki_zerg_description/robot/zerg.urdf.xacro (robot description, xacro)
@@ -12,9 +12,9 @@
   <include filename="$(find gki_sensors_description)/urdf/hokuyo_urg.urdf.xacro" />
   <include filename="$(find gki_sensors_description)/urdf/axis215.urdf.xacro" />
-  <xacro:hokuyo_urg name="base_laser" parent="base_link" ros_topic="base_scan" update_rate="10" ray_count="667" min_angle="120" max_angle="-120">
-    <origin xyz="0.1 0.0 0.138" rpy="0 0 0"/>
+  <xacro:hokuyo_urg name="base_laser" parent="base_link" ros_topic="base_scan" update_rate="30" ray_count="1080" min_angle="135" max_angle="-135">
+    <origin xyz="0.12 0.0 0.178" rpy="0 0 0"/>
   </xacro:hokuyo_urg>
-  <xacro:axis215 name="axis" parent="base_link">
-    <origin xyz="0.0 0.0 0.41" rpy="0 0 0"/>
+  <xacro:axis215 name="axis" parent="bar_horizontal_0_link">
+    <origin xyz="0.0 0.0 0.01" rpy="0 0 0"/>
   </xacro:axis215>
   <joint name="imu_joint" type="fixed">

File: gki_zerg/gki_zerg_description/urdf/zerg_parts.urdf.xacro (robot description, xacro)
@@ -67,4 +67,62 @@
     </link>
   </xacro:macro>
+  <xacro:macro name="bar_side_horizontal" params="parent number x_loc y_loc z_loc">
+    <joint name="bar_side_horizontal_${number}_joint" type="fixed">
+      <origin xyz="${x_loc} ${y_loc} ${z_loc}" rpy="0 0 0"/>
+      <parent link="${parent}"/>
+      <child link="bar_side_horizontal_${number}_link"/>
+    </joint>
+    <link name="bar_side_horizontal_${number}_link">
+      <visual>
+        <origin xyz="0 0 0" rpy="0 0 0"/>
+        <geometry>
+            <box size="0.3 0.04 0.02" />
+        </geometry>
+        <xacro:insert_block name="material_light_grey"/>
+      </visual>
+      <collision>
+        <origin xyz="0 0 0" rpy="0 0 0"/>
+        <geometry>
+            <box size="0.3 0.04 0.02" />
+        </geometry>
+      </collision>
+      <inertial>
+        <mass value="0.01"/>
+        <origin xyz="0 0 0"/>
+        <inertia ixx="0.0001" ixy="0.0" ixz="0.0"
+                 iyy="0.0001" iyz="0.0"
+                 izz="0.0001"/>
+      </inertial>
+    </link>
+  </xacro:macro>
+  <xacro:macro name="cube_holder" params="parent number x_loc y_loc z_loc">
+    <joint name="cube_holder_${number}_joint" type="fixed">
+      <origin xyz="${x_loc} ${y_loc} ${z_loc}" rpy="0 0 0"/>
+      <parent link="${parent}"/>
+      <child link="cube_holder_${number}_link"/>
+    </joint>
+    <link name="cube_holder_${number}_link">
+      <visual>
+        <origin xyz="0 0 0" rpy="0 0 0"/>
+        <geometry>
+            <mesh filename="package://gki_zerg_description/meshes/cube_holder_rviz.stl"/>
+        </geometry>
+        <xacro:insert_block name="material_light_grey"/>
+      </visual>
+      <collision>
+        <origin xyz="0 0 0" rpy="0 0 0"/>
+        <geometry>
+            <mesh filename="package://gki_zerg_description/meshes/cube_holder_rviz.stl"/>
+        </geometry>
+      </collision>
+      <inertial>
+        <mass value="0.01"/>
+        <origin xyz="0 0 0"/>
+        <inertia ixx="0.0001" ixy="0.0" ixz="0.0"
+                 iyy="0.0001" iyz="0.0"
+                 izz="0.0001"/>
+      </inertial>
+    </link>
+  </xacro:macro>
   <!--
     Stack macro - all the components relative transforms are made with respect
@@ -75,5 +133,8 @@
     <bar_vertical parent="${parent}" number="0" x_loc="0.0" y_loc= "0.1885" z_loc="0.2585"/>
     <bar_vertical parent="${parent}" number="1" x_loc="0.0" y_loc="-0.1885" z_loc="0.2585"/>
-    <bar_horizontal parent="${parent}" number="0" x_loc="0.0" y_loc="0.0" z_loc="0.4"/>
+    <bar_horizontal parent="${parent}" number="0" x_loc="-0.17" y_loc="0.0" z_loc="0.41"/>
+    <bar_side_horizontal parent="${parent}" number="0" x_loc="0.0" y_loc="0.1585" z_loc="0.4"/>
+    <bar_side_horizontal parent="${parent}" number="1" x_loc="0.0" y_loc="-0.1585" z_loc="0.4"/>
+    <cube_holder parent="${parent}" number="0" x_loc="0.10" y_loc="0.0" z_loc="0.25"/>
   </xacro:macro>
 </robot>

Commit message: corrected urdf from real robot measurements

File: gki_zerg/gki_zerg_description/robot/zerg.urdf.xacro (robot description, xacro)
@@ -13,5 +13,5 @@
   <include filename="$(find gki_sensors_description)/urdf/axis215.urdf.xacro" />
   <xacro:hokuyo_urg name="base_laser" parent="base_link" ros_topic="base_scan" update_rate="30" ray_count="1080" min_angle="135" max_angle="-135">
-    <origin xyz="0.12 0.0 0.178" rpy="0 0 0"/>
+    <origin xyz="0.12 0.0 0.138" rpy="0 0 0"/>
   </xacro:hokuyo_urg>
   <xacro:axis215 name="axis" parent="bar_horizontal_0_link">

File: gki_zerg/gki_zerg_description/urdf/zerg_parts.urdf.xacro (robot description, xacro)
@@ -96,11 +96,16 @@
     </link>
   </xacro:macro>
-  <xacro:macro name="cube_holder" params="parent number x_loc y_loc z_loc">
-    <joint name="cube_holder_${number}_joint" type="fixed">
-      <origin xyz="${x_loc} ${y_loc} ${z_loc}" rpy="0 0 0"/>
-      <parent link="${parent}"/>
-      <child link="cube_holder_${number}_link"/>
-    </joint>
-    <link name="cube_holder_${number}_link">
+  <xacro:property name="material_tan2">
+    <material name="tan2">
+      <color rgba="0.93 0.60 0.28 1"/>
+    </material>
+  </xacro:property>
+  <xacro:macro name="cube_holder" params="parent x_loc y_loc z_loc">
+    <joint name="cube_holder_joint" type="fixed">
+      <origin xyz="${x_loc} ${y_loc} ${z_loc}" rpy="0 0 0"/>
+      <parent link="${parent}"/>
+      <child link="cube_holder_link"/>
+    </joint>
+    <link name="cube_holder_link">
       <visual>
         <origin xyz="0 0 0" rpy="0 0 0"/>
@@ -108,5 +113,5 @@
             <mesh filename="package://gki_zerg_description/meshes/cube_holder_rviz.stl"/>
         </geometry>
-        <xacro:insert_block name="material_light_grey"/>
+        <xacro:insert_block name="material_tan2"/>
       </visual>
       <collision>
@@ -114,4 +119,62 @@
         <geometry>
             <mesh filename="package://gki_zerg_description/meshes/cube_holder_rviz.stl"/>
+        </geometry>
+      </collision>
+      <inertial>
+        <mass value="0.01"/>
+        <origin xyz="0 0 0"/>
+        <inertia ixx="0.0001" ixy="0.0" ixz="0.0"
+                 iyy="0.0001" iyz="0.0"
+                 izz="0.0001"/>
+      </inertial>
+    </link>
+  </xacro:macro>
+  <xacro:macro name="pilot_bar" params="parent x_loc y_loc z_loc">
+    <joint name="pilot_bar_joint" type="fixed">
+      <origin xyz="${x_loc} ${y_loc} ${z_loc}" rpy="0 0 0"/>
+      <parent link="${parent}"/>
+      <child link="pilot_bar_link"/>
+    </joint>
+    <link name="pilot_bar_link">
+      <visual>
+        <origin xyz="0 0 0" rpy="0 0 0"/>
+        <geometry>
+            <box size="0.02 0.36 0.02" />
+        </geometry>
+        <xacro:insert_block name="material_light_grey"/>
+      </visual>
+      <collision>
+        <origin xyz="0 0 0" rpy="0 0 0"/>
+        <geometry>
+            <box size="0.02 0.36 0.02" />
+        </geometry>
+      </collision>
+      <inertial>
+        <mass value="0.01"/>
+        <origin xyz="0 0 0"/>
+        <inertia ixx="0.0001" ixy="0.0" ixz="0.0"
+                 iyy="0.0001" iyz="0.0"
+                 izz="0.0001"/>
+      </inertial>
+    </link>
+  </xacro:macro>
+  <xacro:macro name="pilot_tip" params="parent x_loc y_loc z_loc">
+    <joint name="pilot_tip_joint" type="fixed">
+      <origin xyz="${x_loc} ${y_loc} ${z_loc}" rpy="0 0 0"/>
+      <parent link="${parent}"/>
+      <child link="pilot_tip_link"/>
+    </joint>
+    <link name="pilot_tip_link">
+      <visual>
+        <origin xyz="0 0 0" rpy="0 0 0"/>
+        <geometry>
+            <box size="0.065 0.04 0.02" />
+        </geometry>
+        <xacro:insert_block name="material_light_grey"/>
+      </visual>
+      <collision>
+        <origin xyz="0 0 0" rpy="0 0 0"/>
+        <geometry>
+            <box size="0.065 0.04 0.02" />
         </geometry>
       </collision>
@@ -133,8 +196,10 @@
     <bar_vertical parent="${parent}" number="0" x_loc="0.0" y_loc= "0.1885" z_loc="0.2585"/>
     <bar_vertical parent="${parent}" number="1" x_loc="0.0" y_loc="-0.1885" z_loc="0.2585"/>
-    <bar_horizontal parent="${parent}" number="0" x_loc="-0.17" y_loc="0.0" z_loc="0.41"/>
-    <bar_side_horizontal parent="${parent}" number="0" x_loc="0.0" y_loc="0.1585" z_loc="0.4"/>
-    <bar_side_horizontal parent="${parent}" number="1" x_loc="0.0" y_loc="-0.1585" z_loc="0.4"/>
-    <cube_holder parent="${parent}" number="0" x_loc="0.10" y_loc="0.0" z_loc="0.25"/>
+    <bar_horizontal parent="${parent}" number="0" x_loc="-0.1275" y_loc="0.0" z_loc="0.405"/>
+    <bar_side_horizontal parent="${parent}" number="0" x_loc="0.0475" y_loc="0.1585" z_loc="0.4"/>
+    <bar_side_horizontal parent="${parent}" number="1" x_loc="0.0475" y_loc="-0.1585" z_loc="0.4"/>
+    <cube_holder parent="${parent}" x_loc="0.15" y_loc="0.0" z_loc="0.27"/>
+    <pilot_bar parent="${parent}" x_loc="0.19" y_loc="0.0" z_loc="0.0625"/>
+    <pilot_tip parent="${parent}" x_loc="0.23" y_loc="0.0" z_loc="0.0625"/>
   </xacro:macro>
 </robot>

Commit message: add front cam to urdf

File: gki_zerg/gki_zerg_description/robot/zerg.urdf.xacro (robot description, xacro)
@@ -12,4 +12,5 @@
   <include filename="$(find gki_sensors_description)/urdf/hokuyo_urg.urdf.xacro" />
   <include filename="$(find gki_sensors_description)/urdf/axis215.urdf.xacro" />
+  <include filename="$(find gki_zerg_description)/urdf/front_cam.urdf.xacro" />
   <xacro:hokuyo_urg name="base_laser" parent="base_link" ros_topic="base_scan" update_rate="30" ray_count="1080" min_angle="135" max_angle="-135">
     <origin xyz="0.12 0.0 0.138" rpy="0 0 0"/>
@@ -18,4 +19,7 @@
     <origin xyz="0.0 0.0 0.01" rpy="0 0 0"/>
   </xacro:axis215>
+  <xacro:front_cam name="front_camera" parent="base_link">
+    <origin xyz="0.225 0.0 0.1" rpy="0 0 0"/>
+  </xacro:front_cam>
   <joint name="imu_joint" type="fixed">
       <origin xyz="0.056 0.062 0.0202" rpy="0 0 0"/>

Commit message: front cam tilted to IRDF

File: gki_zerg/gki_zerg_description/robot/zerg.urdf.xacro (robot description, xacro)
@@ -20,5 +20,5 @@
   </xacro:axis215>
   <xacro:front_cam name="front_camera" parent="base_link">
-    <origin xyz="0.225 0.0 0.1" rpy="0 0 0"/>
+    <origin xyz="0.225 0.0 0.1" rpy="0 -0.262 0"/>
   </xacro:front_cam>
   <joint name="imu_joint" type="fixed">
